Commit message: add depth camera for sim

File: urdf/turtlebot3_waffle_pi.urdf (robot description, URDF)
Before this commit: robot turtlebot3_waffle_pi, 11 links, 10 joints
Links:
- added link camera_depth_optical_frame
Joints:
- added joint camera_depth_joint: type fixed, parent camera_rgb_optical_frame, child camera_depth_optical_frame, origin xyz=0 0 0 rpy=0 0 0

Commit message: update launch

File: urdf/turtlebot3_waffle_pi.urdf (robot description, URDF)
Before this commit: robot turtlebot3_waffle_pi, 12 links, 11 joints
Links:
- added link camera_front_depth_optical_frame
- added link camera_front_link
- added link camera_front_optical_frame
- added link camera_left_depth_optical_frame
- added link camera_left_link
- added link camera_left_optical_frame
- added link camera_right_depth_optical_frame
- added link camera_right_link
- added link camera_right_optical_frame
Joints:
- added joint camera_front_depth_joint: type fixed, parent camera_front_optical_frame, child camera_front_depth_optical_frame, origin xyz=0 0 0 rpy=0 0 0
- added joint camera_front_joint: type fixed, parent base_link, child camera_front_link, origin xyz=0.08 0.0 0.3 rpy=0 0.610 0
- added joint camera_front_optical_joint: type fixed, parent camera_front_link, child camera_front_optical_frame, origin xyz=0 0 0 rpy=-1.57 0 -1.57
- added joint camera_left_depth_joint: type fixed, parent camera_left_optical_frame, child camera_left_depth_optical_frame, origin xyz=0 0 0 rpy=0 0 0
- added joint camera_left_joint: type fixed, parent base_link, child camera_left_link, origin xyz=0.08 0.10 0.3 rpy=0 0.785398 1.5708
- added joint camera_left_optical_joint: type fixed, parent camera_left_link, child camera_left_optical_frame, origin xyz=0 0 0 rpy=-1.57 0 -1.57
- added joint camera_right_depth_joint: type fixed, parent camera_right_optical_frame, child camera_right_depth_optical_frame, origin xyz=0 0 0 rpy=0 0 0
- added joint camera_right_joint: type fixed, parent base_link, child camera_right_link, origin xyz=0.08 -0.10 0.3 rpy=0 0.785398 -1.5708
- added joint camera_right_optical_joint: type fixed, parent camera_right_link, child camera_right_optical_frame, origin xyz=0 0 0 rpy=-1.57 0 -1.57
